Commit message: update base driver

File: src/leo/leo_description/urdf/base/leo_base.urdf (robot description, URDF)
Before this commit: robot leo_base_link, 7 links, 6 joints
Links:
- link body_base_link: geometry collision mesh filename=package://leo_description/meshes/leo/base/test/base_link.STL; visual mesh filename=package://leo_description/meshes/leo/base/test/base_link.STL
